Commit message: prompted bad line following.

File: src/robbie/urdf/robbie.xacro (robot description, xacro)
@@ -14,4 +14,11 @@
   <xacro:include filename="$(find robbie)/urdf/macros.xacro"/>
   <xacro:include filename="$(find robbie)/urdf/materials.xacro"/>
+  <!-- Base link for the robot -->
+  <link name="base_link"/>
+  <joint name="base_to_chassis" type="fixed">
+    <parent link="base_link"/>
+    <child link="chassis"/>
+    <origin xyz="0 0 0" rpy="0 0 0"/>
+  </joint>
   <link name='chassis'>
     <xacro:box_inertial name="chassis" m="${chassis_mass}" x="${chassis_length}" y="${chassis_width}" z="${chassis_height}"/>
@@ -171,9 +178,32 @@
     </plugin>
   </gazebo>
+  <!-- Collision detection for bumper sensors -->
+  <link name="bumper_link">
+    <collision name="bumper_collision">
+      <origin xyz="0 0 0" rpy="0 0 0"/>
+      <geometry>
+        <box size="0.22 0.16 0.06"/>
+      </geometry>
+    </collision>
+  </link>
+  <joint name="bumper_joint" type="fixed">
+    <parent link="chassis"/>
+    <child link="bumper_link"/>
+    <origin xyz="0 0 0"/>
+  </joint>
+  <gazebo reference="bumper_link">
+    <sensor name="bumper_sensor" type="contact">
+      <always_on>true</always_on>
+      <update_rate>10.0</update_rate>
+      <contact>
+        <collision>bumper_collision</collision>
+      </contact>
+    </sensor>
+  </gazebo>
   <gazebo reference="camera_link">
     <sensor type="camera" name="camera1">
       <update_rate>30.0</update_rate>
       <camera name="head">
-        <horizontal_fov>1.3962634</horizontal_fov>
+        <horizontal_fov>1.9198622</horizontal_fov>
         <image>
           <width>800</width>

Commit message: cleaning up workspace.

File: src/robbie/urdf/robbie.xacro (robot description, xacro)
@@ -143,5 +143,5 @@
     <parent link="chassis"/>
     <child link="camera_link"/>
-    <origin xyz="${chassis_length/2} 0 ${chassis_height/2+camera_height/2}"/>
+    <origin xyz="${chassis_length/2} 0 ${chassis_height/2+camera_height/2}" rpy="0 1.2 0"/> <!-- ~69 degree downward tilt - road view only -->
   </joint>
   <gazebo reference="chassis">
@@ -205,5 +205,5 @@
       <update_rate>30.0</update_rate>
       <camera name="head">
-        <horizontal_fov>1.9198622</horizontal_fov>
+        <horizontal_fov>2.9</horizontal_fov> <!-- ~170 degrees -->
         <image>
           <width>800</width>

Commit message: adjusting camera

File: src/robbie/urdf/robbie.xacro (robot description, xacro)
@@ -143,5 +143,5 @@
     <parent link="chassis"/>
     <child link="camera_link"/>
-    <origin xyz="${chassis_length/2} 0 ${chassis_height/2+camera_height/2}" rpy="0 1.2 0"/> <!-- ~69 degree downward tilt - road view only -->
+    <origin xyz="0.095 0 -0.01" rpy="0 0 0"/> <!-- Moved slightly forward, no pitch -->
   </joint>
   <gazebo reference="chassis">
@@ -205,5 +205,5 @@
       <update_rate>30.0</update_rate>
       <camera name="head">
-        <horizontal_fov>2.9</horizontal_fov> <!-- ~170 degrees -->
+        <horizontal_fov>2.094</horizontal_fov> <!-- 120 degrees -->
         <image>
           <width>800</width>

Commit message: switching to imitation learning. First commit.

File: src/robbie/urdf/robbie.xacro (robot description, xacro)
@@ -143,5 +143,5 @@
     <parent link="chassis"/>
     <child link="camera_link"/>
-    <origin xyz="0.095 0 -0.01" rpy="0 0 0"/> <!-- Moved slightly forward, no pitch -->
+    <origin xyz="0.095 0 0.2" rpy="0 0.2 0"/> <!-- Raised up, pitched down -->
   </joint>
   <gazebo reference="chassis">
@@ -205,5 +205,5 @@
       <update_rate>30.0</update_rate>
       <camera name="head">
-        <horizontal_fov>2.094</horizontal_fov> <!-- 120 degrees -->
+        <horizontal_fov>1.396</horizontal_fov> <!-- 80 degrees -->
         <image>
           <width>800</width>

Commit message: using lidar now for a watchdog.

File: src/robbie/urdf/robbie.xacro (robot description, xacro)
@@ -240,3 +240,63 @@
     </sensor>
   </gazebo>
+  <!-- LIDAR Link -->
+  <link name="hokuyo_link">
+    <collision>
+      <origin xyz="0 0 0" rpy="0 0 0"/>
+      <geometry>
+        <box size="0.1 0.1 0.1"/>
+      </geometry>
+    </collision>
+    <visual>
+      <origin xyz="0 0 0" rpy="0 0 0"/>
+      <geometry>
+        <box size="0.1 0.1 0.1"/>
+      </geometry>
+      <material name="hokuyo_material">
+        <color rgba="0.1 0.1 0.1 1"/>
+      </material>
+    </visual>
+    <inertial>
+      <mass value="1e-5" />
+      <origin xyz="0 0 0" rpy="0 0 0"/>
+      <inertia ixx="1e-6" ixy="0" ixz="0" iyy="1e-6" iyz="0" izz="1e-6" />
+    </inertial>
+  </link>
+  <joint name="hokuyo_joint" type="fixed">
+    <axis xyz="0 1 0" />
+    <origin xyz="0.05 0 0.1" rpy="0 0 0"/> <!-- Placed on top of chassis -->
+    <parent link="chassis"/>
+    <child link="hokuyo_link"/>
+  </joint>
+  <gazebo reference="hokuyo_link">
+    <sensor type="ray" name="head_hokuyo_sensor">
+      <pose>0 0 0 0 0 0</pose>
+      <visualize>true</visualize>
+      <update_rate>40</update_rate>
+      <ray>
+        <scan>
+          <horizontal>
+            <samples>720</samples>
+            <resolution>1</resolution>
+            <min_angle>-1.570796</min_angle>
+            <max_angle>1.570796</max_angle>
+          </horizontal>
+        </scan>
+        <range>
+          <min>0.10</min>
+          <max>30.0</max>
+          <resolution>0.01</resolution>
+        </range>
+        <noise>
+          <type>gaussian</type>
+          <mean>0.0</mean>
+          <stddev>0.01</stddev>
+        </noise>
+      </ray>
+      <plugin name="gazebo_ros_head_hokuyo_controller" filename="libgazebo_ros_laser.so">
+        <topicName>/scan</topicName>
+        <frameName>hokuyo_link</frameName>
+      </plugin>
+    </sensor>
+  </gazebo>
 </robot>

Commit message: random commits

File: src/robbie/urdf/robbie.xacro (robot description, xacro)
@@ -5,4 +5,6 @@
   <xacro:property name="camera_height" value="0.01"/>
   <xacro:property name="camera_mass" value="0.01"/>
+  <!-- Side length for new cube camera link -->
+  <xacro:property name="camera_side_length" value="0.02"/>
   <xacro:property name="chassis_width" value="0.15"/>
   <xacro:property name="chassis_length" value="0.2"/>
@@ -98,15 +100,16 @@
     </visual>
   </link>
-  <link name='camera_link'>
-    <xacro:box_inertial name="camera_link" m="${camera_mass}" x="${camera_width}" y="${camera_length}" z="${camera_height}"/>
-    <collision name='camera_link_collision'>
-      <geometry>
-        <box size="${camera_length} ${camera_width} ${camera_height}"/>
-      </geometry>
-    </collision>
-    <visual name='camera_link_visual'>
-      <origin xyz="0 0 0" rpy=" 0 0 0"/>
-      <geometry>
-        <box size="${camera_length} ${camera_width} ${camera_height}"/>
+  <!-- Cube camera link replacement -->
+  <link name='cameraBox'>
+    <xacro:box_inertial name="cameraBox" m="${camera_mass}" x="${camera_side_length}" y="${camera_side_length}" z="${camera_side_length}"/>
+    <collision name='cameraBox_collision'>
+      <geometry>
+        <box size="${camera_side_length} ${camera_side_length} ${camera_side_length}"/>
+      </geometry>
+    </collision>
+    <visual name='cameraBox_visual'>
+      <origin xyz="0 0 0" rpy="0 0 0"/>
+      <geometry>
+        <box size="${camera_side_length} ${camera_side_length} ${camera_side_length}"/>
       </geometry>
     </visual>
@@ -142,11 +145,11 @@
   <joint name="camera_joint" type="fixed">
     <parent link="chassis"/>
-    <child link="camera_link"/>
-    <origin xyz="0.095 0 -0.01" rpy="0 0 0"/> <!-- Moved slightly forward, no pitch -->
+    <child link="cameraBox"/>
+    <origin xyz="0.085 0 0.005" rpy="0 0.3 0"/> <!-- Above chassis center, increased downward pitch to clear interior -->
   </joint>
   <gazebo reference="chassis">
     <material>Gazebo/Orange</material>
   </gazebo>
-  <gazebo reference="camera_link">
+  <gazebo reference="cameraBox">
     <material>Gazebo/Blue</material>
   </gazebo>
@@ -201,9 +204,9 @@
     </sensor>
   </gazebo>
-  <gazebo reference="camera_link">
+  <gazebo reference="cameraBox">
     <sensor type="camera" name="camera1">
       <update_rate>30.0</update_rate>
       <camera name="head">
-        <horizontal_fov>2.094</horizontal_fov> <!-- 120 degrees -->
+        <horizontal_fov>2.4</horizontal_fov> <!-- 180 degrees wide FOV -->
         <image>
           <width>800</width>
@@ -212,5 +215,5 @@
         </image>
         <clip>
-          <near>0.02</near>
+          <near>0.005</near> <!-- Reduced near clip to minimize interior artifact -->
           <far>300</far>
         </clip>
@@ -230,5 +233,5 @@
         <imageTopicName>image_raw</imageTopicName>
         <cameraInfoTopicName>camera_info</cameraInfoTopicName>
-        <frameName>camera_link</frameName>
+        <frameName>cameraBox</frameName>
         <hackBaseline>0.07</hackBaseline>
         <distortionK1>0.0</distortionK1>

Commit message: debugging data collection

File: src/robbie/urdf/robbie.xacro (robot description, xacro)
@@ -245,5 +245,5 @@
       <origin xyz="0 0 0" rpy="0 0 0"/>
       <geometry>
-        <box size="0.1 0.1 0.1"/>
+        <box size="0.03 0.03 0.03"/>
       </geometry>
     </collision>
@@ -251,5 +251,5 @@
       <origin xyz="0 0 0" rpy="0 0 0"/>
       <geometry>
-        <box size="0.1 0.1 0.1"/>
+        <box size="0.03 0.03 0.03"/>
       </geometry>
       <material name="hokuyo_material">

Commit message: realtime factor +  camera adjustment.

File: src/robbie/urdf/robbie.xacro (robot description, xacro)
@@ -143,5 +143,5 @@
     <parent link="chassis"/>
     <child link="camera_link"/>
-    <origin xyz="0.095 0 0.2" rpy="0 0.2 0"/> <!-- Raised up, pitched down -->
+    <origin xyz="0.095 0 0.03" rpy="0 0.2 0"/> <!-- On top of chassis, pitched down slightly -->
   </joint>
   <gazebo reference="chassis">

Commit message: Fix data collector, training script, robot sensors, and add gitignore
- Fixed data collector to properly sync messages and collect valid scan data
- Updated training script to use correct data directory path and filter invalid samples
- Adjusted robot camera and lidar positions (no longer floating)
- Increased camera FOV to 100 degrees
- Set realtime factor to 0.5
- Made lidar box smaller (3cm cube)
- Added .gitignore to exclude training data from git

File: src/robbie/urdf/robbie.xacro (robot description, xacro)
@@ -141,7 +141,7 @@
   </joint>
   <joint name="camera_joint" type="fixed">
-    <parent link="chassis"/>
+    <parent link="hokuyo_link"/>
     <child link="camera_link"/>
-    <origin xyz="0.095 0 0.03" rpy="0 0.2 0"/> <!-- On top of chassis, pitched down slightly -->
+    <origin xyz="0 0 0.02" rpy="0 0 0"/> <!-- Directly on top of lidar, level/horizontal -->
   </joint>
   <gazebo reference="chassis">
@@ -205,5 +205,5 @@
       <update_rate>30.0</update_rate>
       <camera name="head">
-        <horizontal_fov>1.396</horizontal_fov> <!-- 80 degrees -->
+        <horizontal_fov>1.745</horizontal_fov> <!-- 100 degrees (increased from 80) -->
         <image>
           <width>800</width>
@@ -265,5 +265,5 @@
   <joint name="hokuyo_joint" type="fixed">
     <axis xyz="0 1 0" />
-    <origin xyz="0.05 0 0.1" rpy="0 0 0"/> <!-- Placed on top of chassis -->
+    <origin xyz="0.08 0 0.04" rpy="0 0 0"/> <!-- Moved forward on top of chassis -->
     <parent link="chassis"/>
     <child link="hokuyo_link"/>

Commit message: Clueboard reading folder initialized: Inc. Yolo training data

File: src/robbie/urdf/robbie.xacro (robot description, xacro)
@@ -14,4 +14,11 @@
   <xacro:include filename="$(find robbie)/urdf/macros.xacro"/>
   <xacro:include filename="$(find robbie)/urdf/materials.xacro"/>
+  <!-- Base link for the robot -->
+  <link name="base_link"/>
+  <joint name="base_to_chassis" type="fixed">
+    <parent link="base_link"/>
+    <child link="chassis"/>
+    <origin xyz="0 0 0" rpy="0 0 0"/>
+  </joint>
   <link name='chassis'>
     <xacro:box_inertial name="chassis" m="${chassis_mass}" x="${chassis_length}" y="${chassis_width}" z="${chassis_height}"/>
@@ -134,7 +141,7 @@
   </joint>
   <joint name="camera_joint" type="fixed">
-    <parent link="chassis"/>
+    <parent link="hokuyo_link"/>
     <child link="camera_link"/>
-    <origin xyz="${chassis_length/2} 0 ${chassis_height/2+camera_height/2}"/>
+    <origin xyz="0 0 0.02" rpy="0 0 0"/> <!-- Directly on top of lidar, level/horizontal -->
   </joint>
   <gazebo reference="chassis">
@@ -171,9 +178,32 @@
     </plugin>
   </gazebo>
+  <!-- Collision detection for bumper sensors -->
+  <link name="bumper_link">
+    <collision name="bumper_collision">
+      <origin xyz="0 0 0" rpy="0 0 0"/>
+      <geometry>
+        <box size="0.22 0.16 0.06"/>
+      </geometry>
+    </collision>
+  </link>
+  <joint name="bumper_joint" type="fixed">
+    <parent link="chassis"/>
+    <child link="bumper_link"/>
+    <origin xyz="0 0 0"/>
+  </joint>
+  <gazebo reference="bumper_link">
+    <sensor name="bumper_sensor" type="contact">
+      <always_on>true</always_on>
+      <update_rate>10.0</update_rate>
+      <contact>
+        <collision>bumper_collision</collision>
+      </contact>
+    </sensor>
+  </gazebo>
   <gazebo reference="camera_link">
     <sensor type="camera" name="camera1">
       <update_rate>30.0</update_rate>
       <camera name="head">
-        <horizontal_fov>1.3962634</horizontal_fov>
+        <horizontal_fov>2.1</horizontal_fov> <!-- 110 degrees (increased from 100) -->
         <image>
           <width>800</width>
@@ -210,3 +240,63 @@
     </sensor>
   </gazebo>
+  <!-- LIDAR Link -->
+  <link name="hokuyo_link">
+    <collision>
+      <origin xyz="0 0 0" rpy="0 0 0"/>
+      <geometry>
+        <box size="0.03 0.03 0.03"/>
+      </geometry>
+    </collision>
+    <visual>
+      <origin xyz="0 0 0" rpy="0 0 0"/>
+      <geometry>
+        <box size="0.03 0.03 0.03"/>
+      </geometry>
+      <material name="hokuyo_material">
+        <color rgba="0.1 0.1 0.1 1"/>
+      </material>
+    </visual>
+    <inertial>
+      <mass value="1e-5" />
+      <origin xyz="0 0 0" rpy="0 0 0"/>
+      <inertia ixx="1e-6" ixy="0" ixz="0" iyy="1e-6" iyz="0" izz="1e-6" />
+    </inertial>
+  </link>
+  <joint name="hokuyo_joint" type="fixed">
+    <axis xyz="0 1 0" />
+    <origin xyz="0.08 0 0.04" rpy="0 0 0"/> <!-- Moved forward on top of chassis -->
+    <parent link="chassis"/>
+    <child link="hokuyo_link"/>
+  </joint>
+  <gazebo reference="hokuyo_link">
+    <sensor type="ray" name="head_hokuyo_sensor">
+      <pose>0 0 0 0 0 0</pose>
+      <visualize>false</visualize>
+      <update_rate>40</update_rate>
+      <ray>
+        <scan>
+          <horizontal>
+            <samples>720</samples>
+            <resolution>1</resolution>
+            <min_angle>-1.570796</min_angle>
+            <max_angle>1.570796</max_angle>
+          </horizontal>
+        </scan>
+        <range>
+          <min>0.10</min>
+          <max>30.0</max>
+          <resolution>0.01</resolution>
+        </range>
+        <noise>
+          <type>gaussian</type>
+          <mean>0.0</mean>
+          <stddev>0.01</stddev>
+        </noise>
+      </ray>
+      <plugin name="gazebo_ros_head_hokuyo_controller" filename="libgazebo_ros_laser.so">
+        <topicName>scan</topicName>
+        <frameName>hokuyo_link</frameName>
+      </plugin>
+    </sensor>
+  </gazebo>
 </robot>

Commit message: Added 2x 4k cameras to robbie

File: src/robbie/urdf/robbie.xacro (robot description, xacro)
@@ -300,3 +300,93 @@
     </sensor>
   </gazebo>
+  <!-- ============================== -->
+  <!-- LEFT FRONT CAMERA (4K, +30°)   -->
+  <!-- ============================== -->
+  <link name="left_front_cam_link">
+    <inertial>
+      <mass value="0.01"/>
+      <inertia ixx="1e-6" iyy="1e-6" izz="1e-6" ixy="0" ixz="0" iyz="0"/>
+    </inertial>
+    <visual>
+      <geometry>
+        <box size="0.02 0.02 0.01"/>
+      </geometry>
+      <material name="Gazebo/Black"/>
+    </visual>
+  </link>
+  <joint name="left_front_cam_joint" type="fixed">
+    <parent link="chassis"/>
+    <child link="left_front_cam_link"/>
+    <!-- front + left side of chassis, tilted outward -->
+    <origin xyz="${chassis_length/2} 0.05 0.08" rpy="0 0 0.5236"/>
+  </joint>
+  <gazebo reference="left_front_cam_link">
+    <sensor type="camera" name="left_front_camera_sensor">
+      <always_on>true</always_on>
+      <update_rate>30</update_rate>
+      <camera>
+        <horizontal_fov>1.396</horizontal_fov>
+        <image>
+          <width>3840</width>
+          <height>2160</height>
+          <format>R8G8B8</format>
+        </image>
+        <clip>
+          <near>0.02</near>
+          <far>200</far>
+        </clip>
+      </camera>
+      <plugin name="left_front_camera_controller" filename="libgazebo_ros_camera.so">
+        <cameraName>left_front_cam</cameraName>
+        <imageTopicName>left_front/image_raw</imageTopicName>
+        <cameraInfoTopicName>left_front/camera_info</cameraInfoTopicName>
+        <frameName>left_front_cam_link</frameName>
+      </plugin>
+    </sensor>
+  </gazebo>
+  <!-- ============================== -->
+  <!-- RIGHT FRONT CAMERA (4K, -30°)  -->
+  <!-- ============================== -->
+  <link name="right_front_cam_link">
+    <inertial>
+      <mass value="0.01"/>
+      <inertia ixx="1e-6" iyy="1e-6" izz="1e-6" ixy="0" ixz="0" iyz="0"/>
+    </inertial>
+    <visual>
+      <geometry>
+        <box size="0.02 0.02 0.01"/>
+      </geometry>
+      <material name="Gazebo/Black"/>
+    </visual>
+  </link>
+  <joint name="right_front_cam_joint" type="fixed">
+    <parent link="chassis"/>
+    <child link="right_front_cam_link"/>
+    <!-- front + right side of chassis, tilted outward -->
+    <origin xyz="${chassis_length/2} -0.05 0.08" rpy="0 0 -0.5236"/>
+  </joint>
+  <gazebo reference="right_front_cam_link">
+    <sensor type="camera" name="right_front_camera_sensor">
+      <always_on>true</always_on>
+      <update_rate>30</update_rate>
+      <camera>
+        <horizontal_fov>1.396</horizontal_fov>
+        <image>
+          <width>3840</width>
+          <height>2160</height>
+          <format>R8G8B8</format>
+        </image>
+        <clip>
+          <near>0.02</near>
+          <far>200</far>
+        </clip>
+      </camera>
+      <plugin name="right_front_camera_controller" filename="libgazebo_ros_camera.so">
+        <cameraName>right_front_cam</cameraName>
+        <imageTopicName>right_front/image_raw</imageTopicName>
+        <cameraInfoTopicName>right_front/camera_info</cameraInfoTopicName>
+        <frameName>right_front_cam_link</frameName>
+      </plugin>
+    </sensor>
+  </gazebo>
 </robot>

Commit message: Nov. 27 YOLO

File: src/robbie/urdf/robbie.xacro (robot description, xacro)
@@ -319,5 +319,5 @@
     <child link="left_front_cam_link"/>
     <!-- front + left side of chassis, tilted outward -->
-    <origin xyz="${chassis_length/2} 0.05 0.08" rpy="0 0 0.5236"/>
+    <origin xyz="${chassis_length/2} 0.05 0.08" rpy="0 0 0.3491"/>
   </joint>
   <gazebo reference="left_front_cam_link">
@@ -364,5 +364,5 @@
     <child link="right_front_cam_link"/>
     <!-- front + right side of chassis, tilted outward -->
-    <origin xyz="${chassis_length/2} -0.05 0.08" rpy="0 0 -0.5236"/>
+    <origin xyz="${chassis_length/2} -0.05 0.08" rpy="0 0 -0.3491"/>
   </joint>
   <gazebo reference="right_front_cam_link">

Commit message: Added random clueboards gen

File: src/robbie/urdf/robbie.xacro (robot description, xacro)
@@ -301,5 +301,5 @@
   </gazebo>
   <!-- ============================== -->
-  <!-- LEFT FRONT CAMERA (4K, +30°)   -->
+  <!-- LEFT FRONT CAMERA (4K)         -->
   <!-- ============================== -->
   <link name="left_front_cam_link">
@@ -319,5 +319,5 @@
     <child link="left_front_cam_link"/>
     <!-- front + left side of chassis, tilted outward -->
-    <origin xyz="${chassis_length/2} 0.05 0.08" rpy="0 0 0.3491"/>
+    <origin xyz="${chassis_length/2 - 0.1} 0.05 0.08" rpy="0 0 0.3491"/>
   </joint>
   <gazebo reference="left_front_cam_link">
@@ -346,5 +346,5 @@
   </gazebo>
   <!-- ============================== -->
-  <!-- RIGHT FRONT CAMERA (4K, -30°)  -->
+  <!-- RIGHT FRONT CAMERA (4K)        -->
   <!-- ============================== -->
   <link name="right_front_cam_link">
@@ -364,5 +364,5 @@
     <child link="right_front_cam_link"/>
     <!-- front + right side of chassis, tilted outward -->
-    <origin xyz="${chassis_length/2} -0.05 0.08" rpy="0 0 -0.3491"/>
+    <origin xyz="${chassis_length/2 - 0.1} -0.05 0.08" rpy="0 0 -0.3491"/>
   </joint>
   <gazebo reference="right_front_cam_link">
