Commit message: friend working

File: src/robbie/urdf/robbie.xacro (robot description, xacro)
@@ -8,5 +8,5 @@
   <xacro:property name="chassis_length" value="0.2"/>
   <xacro:property name="chassis_height" value="0.05"/>
-  <xacro:property name="chassis_mass" value="0.32"/>
+  <xacro:property name="chassis_mass" value="0.5"/>
   <xacro:property name="wheel_radius" value="0.04"/>
   <xacro:property name="wheel_width" value="0.03"/>
@@ -258,5 +258,5 @@
     </visual>
     <inertial>
-      <mass value="0.01" />
+      <mass value="1e-5" />
       <origin xyz="0 0 0" rpy="0 0 0"/>
       <inertia ixx="1e-6" ixy="0" ixz="0" iyy="1e-6" iyz="0" izz="1e-6" />
@@ -318,5 +318,5 @@
     </visual>
     <inertial>
-      <mass value="0.01" />
+      <mass value="1e-5" />
       <origin xyz="0 0 0" rpy="0 0 0"/>
       <inertia ixx="1e-6" ixy="0" ixz="0" iyy="1e-6" iyz="0" izz="1e-6" />
@@ -339,6 +339,6 @@
             <samples>60</samples>
             <resolution>1</resolution>
-            <min_angle>-0.2705</min_angle>  <!-- -15.5 degrees -->
-            <max_angle>0.2705</max_angle>   <!-- +15.5 degrees (31 degree cone) -->
+            <min_angle>-0.2182</min_angle>  <!-- -12.5 degrees -->
+            <max_angle>0.2182</max_angle>   <!-- +12.5 degrees (25 degree cone) -->
           </horizontal>
         </scan>
@@ -378,5 +378,5 @@
     </visual>
     <inertial>
-      <mass value="0.01" />
+      <mass value="1e-5" />
       <origin xyz="0 0 0" rpy="0 0 0"/>
       <inertia ixx="1e-6" ixy="0" ixz="0" iyy="1e-6" iyz="0" izz="1e-6" />
@@ -438,5 +438,5 @@
     </visual>
     <inertial>
-      <mass value="0.01" />
+      <mass value="1e-5" />
       <origin xyz="0 0 0" rpy="0 0 0"/>
       <inertia ixx="1e-6" ixy="0" ixz="0" iyy="1e-6" iyz="0" izz="1e-6" />
@@ -498,5 +498,5 @@
     </visual>
     <inertial>
-      <mass value="0.01" />
+      <mass value="1e-5" />
       <origin xyz="0 0 0" rpy="0 0 0"/>
       <inertia ixx="1e-6" ixy="0" ixz="0" iyy="1e-6" iyz="0" izz="1e-6" />
@@ -558,5 +558,5 @@
     </visual>
     <inertial>
-      <mass value="0.01" />
+      <mass value="1e-5" />
       <origin xyz="0 0 0" rpy="0 0 0"/>
       <inertia ixx="1e-6" ixy="0" ixz="0" iyy="1e-6" iyz="0" izz="1e-6" />

Commit message: working lidar.

File: src/robbie/urdf/robbie.xacro (robot description, xacro)
@@ -325,5 +325,5 @@
   <joint name="front_lidar_joint" type="fixed">
     <axis xyz="0 1 0" />
-    <origin xyz="0.10 0 -0.01" rpy="0 -0.2 0"/> <!-- Directly on front face, lower, pitched up -->
+    <origin xyz="0.10 0 -0.01" rpy="0 -0.27 0"/> <!-- Directly on front face, lower, pitched up ~15.5 degrees -->
     <parent link="chassis"/>
     <child link="front_lidar_link"/>

Commit message: working with good collision detection

File: src/robbie/urdf/robbie.xacro (robot description, xacro)
@@ -337,8 +337,8 @@
         <scan>
           <horizontal>
-            <samples>70</samples>
+            <samples>500</samples>
             <resolution>1</resolution>
-            <min_angle>-0.3054</min_angle>  <!-- -17.5 degrees -->
-            <max_angle>0.3054</max_angle>   <!-- +17.5 degrees (35 degree cone) -->
+            <min_angle>-0.4200</min_angle>  <!-- -27.5 degrees -->
+            <max_angle>0.4200</max_angle>   <!-- +27.5 degrees (55 degree plane) -->
           </horizontal>
         </scan>
@@ -392,13 +392,13 @@
     <sensor type="ray" name="left_lidar_sensor">
       <pose>0 0 0 0 0 0</pose>
-      <visualize>false</visualize>
+      <visualize>true</visualize>
       <update_rate>40</update_rate>
       <ray>
         <scan>
           <horizontal>
-            <samples>15</samples> <!-- 15 degrees scan -->
+            <samples>150</samples> <!-- 45 degrees scan, 5x resolution -->
             <resolution>1</resolution>
             <min_angle>0.2618</min_angle>   <!-- 15 degrees -->
-            <max_angle>0.5236</max_angle>   <!-- 30 degrees -->
+            <max_angle>1.0472</max_angle>   <!-- 60 degrees -->
           </horizontal>
         </scan>
@@ -452,12 +452,12 @@
     <sensor type="ray" name="right_lidar_sensor">
       <pose>0 0 0 0 0 0</pose>
-      <visualize>false</visualize>
+      <visualize>true</visualize>
       <update_rate>40</update_rate>
       <ray>
         <scan>
           <horizontal>
-            <samples>15</samples> <!-- 15 degrees scan -->
+            <samples>150</samples> <!-- 45 degrees scan, 5x resolution -->
             <resolution>1</resolution>
-            <min_angle>-0.5236</min_angle>  <!-- -30 degrees -->
+            <min_angle>-1.0472</min_angle>  <!-- -60 degrees -->
             <max_angle>-0.2618</max_angle>  <!-- -15 degrees -->
           </horizontal>
@@ -512,10 +512,10 @@
     <sensor type="ray" name="side_left_lidar_sensor">
       <pose>0 0 0 0 0 0</pose>
-      <visualize>false</visualize>
+      <visualize>true</visualize>
       <update_rate>40</update_rate>
       <ray>
         <scan>
           <horizontal>
-            <samples>60</samples>
+            <samples>300</samples>
             <resolution>1</resolution>
             <min_angle>-0.523599</min_angle> <!-- -30 degrees -->
@@ -572,10 +572,10 @@
     <sensor type="ray" name="side_right_lidar_sensor">
       <pose>0 0 0 0 0 0</pose>
-      <visualize>false</visualize>
+      <visualize>true</visualize>
       <update_rate>40</update_rate>
       <ray>
         <scan>
           <horizontal>
-            <samples>60</samples>
+            <samples>300</samples>
             <resolution>1</resolution>
             <min_angle>-0.523599</min_angle> <!-- -30 degrees -->
@@ -669,16 +669,16 @@
     <parent link="camera_mount_crossbar"/>
     <child link="left_front_cam_link"/>
-    <!-- Attached to left end of crossbar, tilted outward -->
-    <origin xyz="0 0.05 0" rpy="0 0 0.3491"/>
+    <!-- Attached to left end of crossbar, tilted outward (10 degrees) -->
+    <origin xyz="0 0.05 0" rpy="0 0 0.1746"/>
   </joint>
   <gazebo reference="left_front_cam_link">
     <sensor type="camera" name="left_front_camera_sensor">
       <always_on>true</always_on>
-      <update_rate>30</update_rate>
+      <update_rate>10</update_rate>
       <camera>
         <horizontal_fov>1.396</horizontal_fov>
         <image>
-          <width>3840</width>
-          <height>2160</height>
+          <width>1920</width>
+          <height>1080</height>
           <format>R8G8B8</format>
         </image>
@@ -712,16 +712,16 @@
     <parent link="camera_mount_crossbar"/>
     <child link="right_front_cam_link"/>
-    <!-- Attached to right end of crossbar, tilted outward -->
-    <origin xyz="0 -0.05 0" rpy="0 0 -0.3491"/>
+    <!-- Attached to right end of crossbar, tilted outward (10 degrees) -->
+    <origin xyz="0 -0.05 0" rpy="0 0 -0.1746"/>
   </joint>
   <gazebo reference="right_front_cam_link">
     <sensor type="camera" name="right_front_camera_sensor">
       <always_on>true</always_on>
-      <update_rate>30</update_rate>
+      <update_rate>10</update_rate>
       <camera>
         <horizontal_fov>1.396</horizontal_fov>
         <image>
-          <width>3840</width>
-          <height>2160</height>
+          <width>1920</width>
+          <height>1080</height>
           <format>R8G8B8</format>
         </image>

Commit message: ella-debug camera settings.

File: src/robbie/urdf/robbie.xacro (robot description, xacro)
@@ -669,16 +669,16 @@
     <parent link="camera_mount_crossbar"/>
     <child link="left_front_cam_link"/>
-    <!-- Attached to left end of crossbar, tilted outward (10 degrees) -->
-    <origin xyz="0 0.05 0" rpy="0 0 0.1746"/>
+    <!-- Attached to left end of crossbar, tilted outward -->
+    <origin xyz="0 0.05 0" rpy="0 0 0.3491"/>
   </joint>
   <gazebo reference="left_front_cam_link">
     <sensor type="camera" name="left_front_camera_sensor">
       <always_on>true</always_on>
-      <update_rate>10</update_rate>
+      <update_rate>15</update_rate>
       <camera>
         <horizontal_fov>1.396</horizontal_fov>
         <image>
-          <width>1920</width>
-          <height>1080</height>
+          <width>1280</width>
+          <height>720</height>
           <format>R8G8B8</format>
         </image>
@@ -712,16 +712,16 @@
     <parent link="camera_mount_crossbar"/>
     <child link="right_front_cam_link"/>
-    <!-- Attached to right end of crossbar, tilted outward (10 degrees) -->
-    <origin xyz="0 -0.05 0" rpy="0 0 -0.1746"/>
+    <!-- Attached to right end of crossbar, tilted outward -->
+    <origin xyz="0 -0.05 0" rpy="0 0 -0.3491"/>
   </joint>
   <gazebo reference="right_front_cam_link">
     <sensor type="camera" name="right_front_camera_sensor">
       <always_on>true</always_on>
-      <update_rate>10</update_rate>
+      <update_rate>15</update_rate>
       <camera>
         <horizontal_fov>1.396</horizontal_fov>
         <image>
-          <width>1920</width>
-          <height>1080</height>
+          <width>1280</width>
+          <height>720</height>
           <format>R8G8B8</format>
         </image>

Commit message: done lf for now.

File: src/robbie/urdf/robbie.xacro (robot description, xacro)
@@ -325,5 +325,5 @@
   <joint name="front_lidar_joint" type="fixed">
     <axis xyz="0 1 0" />
-    <origin xyz="0.10 0 -0.01" rpy="0 -0.27 0"/> <!-- Directly on front face, lower, pitched up ~15.5 degrees -->
+    <origin xyz="0.10 0 0.0" rpy="0 -0.25 0"/> <!-- Directly on front face, pitched up ~15.5 degrees -->
     <parent link="chassis"/>
     <child link="front_lidar_link"/>
@@ -332,10 +332,10 @@
     <sensor type="ray" name="front_lidar_sensor">
       <pose>0 0 0 0 0 0</pose>
-      <visualize>false</visualize>
+      <visualize>true</visualize>
       <update_rate>40</update_rate>
       <ray>
         <scan>
           <horizontal>
-            <samples>500</samples>
+            <samples>300</samples>
             <resolution>1</resolution>
             <min_angle>-0.3800</min_angle>  <!-- -27.5 degrees -->
@@ -385,5 +385,5 @@
   <joint name="left_lidar_joint" type="fixed">
     <axis xyz="0 1 0" />
-    <origin xyz="0.10 0.0375 -0.01" rpy="0 -0.2 0"/> <!-- On front face, 1/4 from left edge, angled up -->
+    <origin xyz="0.10 0.0375 0.0" rpy="0 -0.25 0"/> <!-- On front face, 1/4 from left edge, pitched up ~15.5 degrees -->
     <parent link="chassis"/>
     <child link="left_lidar_link"/>
@@ -392,18 +392,18 @@
     <sensor type="ray" name="left_lidar_sensor">
       <pose>0 0 0 0 0 0</pose>
-      <visualize>false</visualize>
+      <visualize>true</visualize>
       <update_rate>40</update_rate>
       <ray>
         <scan>
           <horizontal>
-            <samples>150</samples> <!-- 45 degrees scan, 5x resolution -->
+            <samples>300</samples> <!-- 45 degrees scan, 5x resolution -->
             <resolution>1</resolution>
-            <min_angle>0.2618</min_angle>   <!-- 15 degrees -->
-            <max_angle>1.0472</max_angle>   <!-- 60 degrees -->
+            <min_angle>0.17</min_angle>   <!-- 15 degrees -->
+            <max_angle>1.1</max_angle>   <!-- 60 degrees -->
           </horizontal>
         </scan>
         <range>
-          <min>0.02</min>
-          <max>0.75</max>
+          <min>0.035</min>
+          <max>0.5</max>
           <resolution>0.005</resolution>
         </range>
@@ -445,5 +445,5 @@
   <joint name="right_lidar_joint" type="fixed">
     <axis xyz="0 1 0" />
-    <origin xyz="0.10 -0.0375 -0.01" rpy="0 -0.2 0"/> <!-- On front face, 1/4 from right edge, angled up -->
+    <origin xyz="0.10 -0.0375 0.0" rpy="0 -0.25 0"/> <!-- On front face, 1/4 from right edge, pitched up ~15.5 degrees -->
     <parent link="chassis"/>
     <child link="right_lidar_link"/>
@@ -452,18 +452,18 @@
     <sensor type="ray" name="right_lidar_sensor">
       <pose>0 0 0 0 0 0</pose>
-      <visualize>false</visualize>
+      <visualize>true</visualize>
       <update_rate>40</update_rate>
       <ray>
         <scan>
           <horizontal>
-            <samples>150</samples> <!-- 45 degrees scan, 5x resolution -->
+            <samples>300</samples> <!-- 45 degrees scan, 5x resolution -->
             <resolution>1</resolution>
-            <min_angle>-1.0472</min_angle>  <!-- -60 degrees -->
-            <max_angle>-0.2618</max_angle>  <!-- -15 degrees -->
+            <min_angle>-1.1</min_angle>  <!-- -60 degrees -->
+            <max_angle>-0.17</max_angle>  <!-- -15 degrees -->
           </horizontal>
         </scan>
         <range>
-          <min>0.02</min>
-          <max>0.75</max>
+          <min>0.035</min>
+          <max>0.5</max>
           <resolution>0.005</resolution>
         </range>
